File: V5/EMG_CHANNEL_2_ANALOG.kicad_sch (KiCad schematic)
At the start: 38 parts, among them J401 AudioJack3 TRS, U401 INA333xxDGK, U402 MCP6004

Commit message: fix channel trs mapping and raw gain input polarity
Connections:
- net EMG2_IN_P: now also J401.S; no longer J401.T
- net EMG2_RAW_GAIN_FB: now also U402.3 (+); no longer U402.2 (-)
- net EMG2_RAW_HPF_NODE: now also U402.2 (-); no longer U402.3 (+)
- net EMG2_REF_ELECTRODE: now also J401.T; no longer J401.S
Changed lines of the file:
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@@
 		)
 	)
-	(label "EMG2_REF_ELECTRODE"
+	(label "EMG2_IN_P"
 		(at 38.1 66.04 0)
 		(effects
@@
 		)
 	)
-	(label "EMG2_IN_P"
+	(label "EMG2_REF_ELECTRODE"
 		(at 38.1 71.12 0)
 		(effects
@@
 		)
 	)
+	(label "EMG2_RAW_HPF_NODE"
+		(at 304.8 76.2 180)
+		(effects
+			(font
+				(size 1.27 1.27)
+			)
+			(justify right)
+		)
+	)
 	(label "EMG2_RAW_GAIN_FB"
-		(at 304.8 76.2 180)
-		(effects
-			(font
-				(size 1.27 1.27)
-			)
-			(justify right)
-		)
-	)
-	(label "EMG2_RAW_HPF_NODE"
 		(at 304.8 71.12 180)
 		(effects
