File: V5/EMG_CHANNEL_2_ANALOG.kicad_sch (KiCad schematic)
At the start: 38 parts, among them J401 SJ1-3523N, U401 INA333AIDGKT, U402 MCP6004-I/SL

Commit message: Complete V5 PCB placement and debug access
Parts:
- added TP401: EMG2_IA_OUT, TestPoint:TestPoint_Pad_D1.5mm, symbol Connector:TestPoint
- added TP402: EMG2_RAW_DRV, TestPoint:TestPoint_Pad_D1.5mm, symbol Connector:TestPoint
- added TP403: EMG2_RECT_DRV, TestPoint:TestPoint_Pad_D1.5mm, symbol Connector:TestPoint
- added TP404: EMG2_ENV_DRV, TestPoint:TestPoint_Pad_D1.5mm, symbol Connector:TestPoint
- added TP405: GND_CH2, TestPoint:TestPoint_Pad_D2.0mm, symbol Connector:TestPoint
Connections:
- net EMG2_ENV_DRV: now also TP404.1
- net EMG2_IA_OUT: now also TP401.1
- net EMG2_RAW_DRV: now also TP402.1
- net EMG2_RECT_DRV: now also TP403.1
- net GND: now also TP405.1

Commit message: Update V5 routing and INA333 footprint
Parts:
- U401: footprint Package_SO:VSSOP-8_3x3mm_P0.65mm -> EMG_V5:INA333_DGK_VSSOP-8_TI
Changed lines of the file:
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@@
 			)
 		)
-		(property "Footprint" "Package_SO:VSSOP-8_3x3mm_P0.65mm"
+		(property "Footprint" "EMG_V5:INA333_DGK_VSSOP-8_TI"
 			(at 210.82 73.66 0)
 			(hide yes)
