File: V5/POWER_REFERENCE_BLOCK.kicad_sch (KiCad schematic)
At the start: 45 parts, among them J201 B2B-XH-A(LF)(SN), Q201 PMV48XP, SW201 TS02CQE, U201 MCP3208-CI/P, U202 MCP6002-I/SN, U203 TPS7A2033PDBVR, U204 TPS22917DBVR, U205 TXU0304PWR, U206 TPS3899DL30DSER, U207 TPS3899DL29DSER

Commit message: assign final resistor footprints
Parts:
- R201, R202, R204, R205: footprint (none) -> Resistor_SMD:R_0805_2012Metric
Changed lines of the file:
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@@
 			)
 		)
-		(property "Footprint" ""
+		(property "Footprint" "Resistor_SMD:R_0805_2012Metric"
 			(at 43.18 161.29 0)
 			(show_name no)
@@
 			)
 		)
-		(property "Footprint" ""
+		(property "Footprint" "Resistor_SMD:R_0805_2012Metric"
 			(at 43.18 176.53 0)
 			(show_name no)
@@
 			)
 		)
-		(property "Footprint" ""
+		(property "Footprint" "Resistor_SMD:R_0805_2012Metric"
 			(at 269.24 104.14 0)
 			(show_name no)
@@
 			)
 		)
-		(property "Footprint" ""
+		(property "Footprint" "Resistor_SMD:R_0805_2012Metric"
 			(at 269.24 119.38 0)
 			(show_name no)

Commit message: Assign Murata GRM32 footprint and update C213 to 47uF
Parts:
- C213: value 22uF -> 47uF; footprint (none) -> EMG_V5:C_1210_3225_Murata_GRM32_Reflow
Changed lines of the file:
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@@
 			)
 		)
-		(property "Value" "22uF"
+		(property "Value" "47uF"
 			(at 236.474 63.5 0)
 			(show_name no)
@@
 			)
 		)
-		(property "Footprint" ""
+		(property "Footprint" "EMG_V5:C_1210_3225_Murata_GRM32_Reflow"
 			(at 232.105 66.04 0)
 			(hide yes)
