File: V5/EMG_CHANNEL_1_ANALOG.kicad_sch (KiCad schematic)
At the start: 38 parts, among them J301 SJ1-3523N, U301 INA333AIDGKT, U302 MCP6004-I/SL

Commit message: Complete V5 PCB placement and debug access
Parts:
- added TP301: EMG1_IA_OUT, TestPoint:TestPoint_Pad_D1.5mm, symbol Connector:TestPoint
- added TP302: EMG1_RAW_DRV, TestPoint:TestPoint_Pad_D1.5mm, symbol Connector:TestPoint
- added TP303: EMG1_RECT_DRV, TestPoint:TestPoint_Pad_D1.5mm, symbol Connector:TestPoint
- added TP304: EMG1_ENV_DRV, TestPoint:TestPoint_Pad_D1.5mm, symbol Connector:TestPoint
- added TP305: GND_CH1, TestPoint:TestPoint_Pad_D2.0mm, symbol Connector:TestPoint
- added TP306: ANALOG_VREF, TestPoint:TestPoint_Pad_D1.5mm, symbol Connector:TestPoint
Connections:
- net EMG1_ENV_DRV: now also TP304.1
- net EMG1_IA_OUT: now also TP301.1
- net EMG1_RAW_DRV: now also TP302.1
- net EMG1_RECT_DRV: now also TP303.1
- net GND: now also TP305.1
- net analog VREF: now also TP306.1

Commit message: Update V5 routing and INA333 footprint
Parts:
- U301: footprint Package_SO:VSSOP-8_3x3mm_P0.65mm -> EMG_V5:INA333_DGK_VSSOP-8_TI
Changed lines of the file:
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@@
 			)
 		)
-		(property "Footprint" "Package_SO:VSSOP-8_3x3mm_P0.65mm"
+		(property "Footprint" "EMG_V5:INA333_DGK_VSSOP-8_TI"
 			(at 210.82 73.66 0)
 			(hide yes)
